Commit message: feat: Add mock hardware and MoveIt config
- Add mock_components/GenericSystem xacro for hardware-free simulation
- Add mock controller configs (JTC with position interface)
- Add mock launch files for standalone testing
- Add MoveIt config package (SRDF, kinematics, OMPL, controllers)
- Add MoveIt launch files with use_mock parameter (mock/real hardware)
- Add RViz config with MotionPlanning plugin

File: dg5f_s_driver/urdf/dg5f_s_15dof_left_ros2_control.xacro (robot description, xacro)
@@ -42,5 +42,12 @@
         </joint>
     </xacro:if>
-    <!-- ROS2 Control -->
+    <!-- Dummy base_link for KDL compatibility -->
+    <link name="base_link" />
+    <joint name="base_joint" type="fixed">
+        <parent link="base_link" />
+        <child link="link_base" />
+        <origin xyz="0 0 0" rpy="0 0 0" />
+    </joint>
+        <!-- ROS2 Control -->
     <ros2_control name="DG5FS15DofLeftHardware" type="system">
         <hardware>

File: dg5f_s_driver/urdf/dg5f_s_15dof_right_ros2_control.xacro (robot description, xacro)
@@ -42,5 +42,12 @@
         </joint>
     </xacro:if>
-    <!-- ROS2 Control -->
+    <!-- Dummy base_link for KDL compatibility -->
+    <link name="base_link" />
+    <joint name="base_joint" type="fixed">
+        <parent link="base_link" />
+        <child link="link_base" />
+        <origin xyz="0 0 0" rpy="0 0 0" />
+    </joint>
+        <!-- ROS2 Control -->
     <ros2_control name="DG5FS15DofRightHardware" type="system">
         <hardware>

File: dg5f_s_driver/urdf/dg5f_s_left_ros2_control.xacro (robot description, xacro)
@@ -42,5 +42,12 @@
         </joint>
     </xacro:if>
-    <!-- ROS2 Control -->
+    <!-- Dummy base_link for KDL compatibility -->
+    <link name="base_link" />
+    <joint name="base_joint" type="fixed">
+        <parent link="base_link" />
+        <child link="link_base" />
+        <origin xyz="0 0 0" rpy="0 0 0" />
+    </joint>
+        <!-- ROS2 Control -->
     <ros2_control name="DG5FSLeftHardware" type="system">
         <hardware>

File: dg5f_s_driver/urdf/dg5f_s_right_ros2_control.xacro (robot description, xacro)
@@ -42,5 +42,12 @@
         </joint>
     </xacro:if>
-    <!-- ROS2 Control -->
+    <!-- Dummy base_link for KDL compatibility -->
+    <link name="base_link" />
+    <joint name="base_joint" type="fixed">
+        <parent link="base_link" />
+        <child link="link_base" />
+        <origin xyz="0 0 0" rpy="0 0 0" />
+    </joint>
+        <!-- ROS2 Control -->
     <ros2_control name="DG5FSRightHardware" type="system">
         <hardware>
